File: hardware/hv_sense/hv_sense.kicad_pcb (KiCad board)
At the start: 2 copper layers, 94.4 x 70.7 mm, 71 parts, among them J1 Conn_01x02, J2 Conn_01x06, J3 Conn_01x04, J6 Conn_01x02, J7 Conn_01x06, U1 4081, U10 140817141410, U2 4071, U3 4081, U4 40106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

Commit message: Added switch to comply with FSUK rules
Parts:
- added SW1: SW_SPDT, Connector_PinHeader_2.54mm:PinHeader_1x03_P2.54mm_Vertical, F.Cu at (152.9, 52.6)
- moved C8 2.73 mm to (152.4, 46.5)
Connections:
- net /Implausibility and LED logic/TS_UNSAFE renamed Net-(U2-Pad5)
- net Net-(U1-Pad11) renamed /Implausibility and LED logic/~{TSAL_ACTIVE}
- D5 pad 1: /~{HV_DETECTED} -> Net-(D5-Pad1)
Routing:
- net /~{HV_DETECTED}: track 48.0 -> 34.3 mm, vias 4 -> 3
- net /Implausibility and LED logic/~{TSAL_ACTIVE}: track 53.5 -> 67.1 mm, vias 2 -> 4
- net Net-(D5-Pad1): track 0.00 -> 6.85 mm
- net /Implausibility and LED logic/RED_LED_ON: track 37.5 -> 35.8 mm
- net /~{HIGH_AIR_MECH_ON}: track 83.1 -> 83.8 mm
- net +12V: track 266.1 -> 265.4 mm
- net /~{LOW_AIR_MECH_ON}: track 81.0 -> 81.6 mm

Commit message: Added PCB updates
Parts:
- added R30: 82, Resistor_SMD:R_2512_6332Metric, F.Cu at (173.3, 27.1)
- added R31: 82, Resistor_SMD:R_2512_6332Metric, F.Cu at (182.2, 27.1)
- added R32: 82, Resistor_SMD:R_2512_6332Metric, F.Cu at (173.3, 31.5)
- PS1: value MPWF1212S-3W -> 0.5S7B_1212S3UP; footprint footprints:MPWF1212S-3W -> footprints:0.5S7B_1212S3UP
- R1: value 10k -> 82; footprint Resistor_SMD:R_0603_1608Metric -> Resistor_SMD:R_2512_6332Metric
- moved R1 30.8 mm to (182.2, 31.5), turned to 180 degrees
- moved H2 13.7 mm to (196.4, 29.1)
- moved PS1 8.36 mm to (133.3, 36.3), turned to 180 degrees
- moved J2 8.00 mm to (163.0, 30.2)
- moved J6 5.28 mm to (194.7, 39.9)
Connections:
- PS1 pad 1: GND -> +12V
- PS1 pad 2: +12V -> GND
- PS1 pad 5: (no net) -> /HV_GND
- PS1 pad 7: /HV_GND -> /HV_+12V
- R1 pad 1: /~{PRCHG_MECH_ON} -> +12V
- R1 pad 2: +12V -> Net-(R1-Pad2)
Routing:
- net /~{PRCHG_MECH_ON}: track 71.6 -> 90.3 mm
- net +12V: track 265.4 -> 279.2 mm, vias 8 -> 6
- net GND: track 55.3 -> 68.3 mm
- net Net-(R1-Pad2): track 0.00 -> 10.4 mm
- net /HV_GND: track 80.3 -> 88.9 mm
- net /~{HIGH_AIR_MECH_ON}: track 83.8 -> 75.8 mm
- net /HV_+12V: track 79.2 -> 75.8 mm
- net /~{LOW_AIR_MECH_ON}: track 81.6 -> 84.4 mm
- net /Implausibility and LED logic/~{TSAL_ACTIVE}: track 67.1 -> 65.8 mm
