File: hardware/hv_sense/logic.kicad_sch (KiCad schematic)
At the start: 32 parts, among them U1 4081, U2 4071, U3 4081, U4 40106, U5 40106, U6 4013

Commit message: Changed connector footprints
Other:
- company: (none) -> SUFST - Southampton University Formula Student Team
- title: (none) -> TSAL Sense / Logic - Implausibility Check
Changed lines of the file:
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@@
 (kicad_sch (version 20211123) (generator eeschema)
   (paper "A3")
+  (title_block
+    (title "TSAL Sense / Logic - Implausibility Check")
+    (date "2022-04-01")
+    (rev "1")
+    (company "SUFST - Southampton University Formula Student Team")
+  )
   (junction (at 116.205 79.375) (diameter 0) (color 0 0 0 0)
   )

Commit message: Added switch to comply with FSUK rules
Parts:
- added SW1: (no value), symbol Switch:SW_SPDT
Connections:
- net ~{HV_DETECTED}: now also SW1.3 (C); no longer D5.1 (A)
- net ~{TSAL_ACTIVE}: now reaches U1.11, U5.9
- net ~{TSAL_ACTIVE}: now also SW1.1 (A)
- net TS_UNSAFE: no longer names the net of U2.5, U5.8
- new net: D5.1 (A), SW1.2 (B)
Other:
- note added: "FSG rules"
- note added: "FSUK rules"
- note added: "GREEN_LED_ON - true unless TSAL_ACTIVE or IMPLAUSIBLE."
- note removed: "GREEN_LED_ON - true unless TS_UNSAFE or IMPLAUSIBLE."
- note removed: "TS_UNSAFE - relay closed or HV measured."

Commit message: Added PCB updates
Parts:
- SW1: value (none) -> SW_SPDT; footprint (none) -> Connector_PinHeader_2.54mm:PinHeader_1x03_P2.54mm_Vertical
Changed lines of the file:
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@@
     (in_bom yes) (on_board yes) (fields_autoplaced)
     (property "Reference" "SW1" (id 0) (at 196.215 113.03 0))
-    (property "Value" "" (id 1) (at 196.215 115.57 0))
-    (property "Footprint" "" (id 2) (at 196.215 121.285 0)
+    (property "Value" "SW_SPDT" (id 1) (at 196.215 115.57 0))
+    (property "Footprint" "Connector_PinHeader_2.54mm:PinHeader_1x03_P2.54mm_Vertical" (id 2) (at 196.215 121.285 0)
       (effects (font (size 1.27 1.27)) hide)
     )
